File: design/jetson-minimal.kicad_sch (KiCad schematic)
At the start: 92 parts, among them J1 SI-51005-F, J2 RJ45_RB1-125B8G1A, J3 Jack-DC, J4 power in, J5 2309414-1, J6 Conn_01x04_Male, J7 USB_C_Receptacle, J8 PROG, J9 reset, Q1 DMN26D0UT-7, Q2 DMN26D0UT-7, Q3 DMN26D0UT-7, Q4 DMN26D0UT-7, Q5 DMN26D0UT-7, Q6 DMN26D0UT-7, U1 74LVC1G126, U2 TLV62569DDC, U3 TLV70018DCKT, U4 74LVC1G126

Commit message: updaed some compoent footprints and layouts to make it easier for manufacturing
Parts:
- J3: now fitted
- J4: now not fitted
- R1, R10, R11, R12, R14, R15, R16, R19, R20, R29, R32, R34, R6, R8, R9: footprint Resistor_SMD:R_0402_1005Metric -> Resistor_SMD:R_0603_1608Metric_Pad0.98x0.95mm_HandSolder; Package 0402 -> 0603
- R13, R18, R21, R30, R31, R33, R4, R5, R7: footprint Resistor_SMD:R_0402_1005Metric -> Resistor_SMD:R_0603_1608Metric_Pad0.98x0.95mm_HandSolder
- R17: footprint Resistor_SMD:R_0603_1608Metric -> Resistor_SMD:R_0603_1608Metric_Pad0.98x0.95mm_HandSolder
- R35: value 1M -> 100k; footprint Resistor_SMD:R_0402_1005Metric -> Resistor_SMD:R_0603_1608Metric_Pad0.98x0.95mm_HandSolder
- R36, R37: footprint Resistor_SMD:R_0402_1005Metric -> Resistor_SMD:R_0603_1608Metric_Pad0.98x0.95mm_HandSolder; Package 0402 -> 0603; now not fitted; now left out of the parts list
- U5: now not fitted; now left out of the parts list
Other:
- moved on the sheet: C1, C3
