File: design/Page12.kicad_sch (KiCad schematic)
At the start: 0 parts

Commit message: updated, its functional, but needs routing finished. tweeks from Bornhack 2026 to be added. :)
Parts:
- added C48, C49, C50, C51, C52, C53, C54, C55, C56: 0.1uF, Capacitor_SMD:C_0805_2012Metric_Pad1.18x1.45mm_HandSolder, symbol Device:C
- added J11: HDMI_A, Libraries:HDMI_A_Amphenol_10029449-111, symbol Connector:HDMI_A
- added Q11, Q13: DMN26D0UT-7, Package_TO_SOT_SMD:SOT-523, symbol Transistor_FET:2N7002
- added R59, R60, R61, R62, R63, R64, R65, R66: 510r, Resistor_SMD:R_0805_2012Metric_Pad1.20x1.40mm_HandSolder, symbol Device:R
- added R71, R72, R77, R78: 12k, Resistor_SMD:R_0805_2012Metric_Pad1.20x1.40mm_HandSolder, symbol Device:R
Connections:
- new net +3V3_HDMI: C56.1, Q11.1 (G), Q13.1 (G), R71.1, R72.1
- new net +5V_HDMI: J11.18 (+5V), R77.2, R78.2
- new net GND: C56.2, J11.11 (CKS), J11.17 (GND), J11.2 (D2S), J11.5 (D1S), J11.8 (D0S), J11.SH, R59.2, R60.2, R61.2, R62.2, R63.2, R64.2, R65.2, R66.2
- new net HDMI_CEC_CON: J11.13 (CEC)
- new net HDMI_DDC_SCL_POL: Q11.2 (S), R71.2
- new net HDMI_DDC_SCL_POL_CON: J11.15 (SCL), Q11.3 (D), R77.1
- new net HDMI_DDC_SDA_POL: Q13.2 (S), R72.2
- new net HDMI_DDC_SDA_POL_CON: J11.16 (SDA), Q13.3 (D), R78.1
- new net HDMI_HPD_CON: J11.19 (HPD)
- new net HDMI_TX0_CON_N: C54.1, J11.9 (D0-), R61.1
- new net HDMI_TX0_CON_P: C50.1, J11.7 (D0+), R62.1
- new net HDMI_TX1_CON_N: C53.1, J11.6 (D1-), R63.1
- new net HDMI_TX1_CON_P: C49.1, J11.4 (D1+), R64.1
- new net HDMI_TX2_CON_N: C52.1, J11.3 (D2-), R65.1
- new net HDMI_TX2_CON_P: C48.1, J11.1 (D2+), R66.1
- new net HDMI_TXC_CON_N: C55.1, J11.12 (CK-), R59.1
- new net HDMI_TXC_CON_P: C51.1, J11.10 (CK+), R60.1
- new net HDMI_TXC_N: C55.2
- new net HDMI_TXC_P: C51.2
- new net HDMI_TXD0_N: C54.2
- new net HDMI_TXD0_P: C50.2
- new net HDMI_TXD1_N: C53.2
- new net HDMI_TXD1_P: C49.2
- new net HDMI_TXD2_N: C52.2
- new net HDMI_TXD2_P: C48.2
- no-connect marks 0 -> 1
Other:
- note added: "DNP for MPV"
- note added: "HDMI CONNECTIONS"
- note added: "No stuff the common mode choke, co-locate resistors to avoid stubs"
- note added: "short. and remove."
