File: design/Page4.kicad_sch (KiCad schematic)
At the start: 10 parts, among them J5 2309414-1, Q6 DMN26D0UT-7, Q7 DMN26D0UT-7

Commit message: updated, its functional, but needs routing finished. tweeks from Bornhack 2026 to be added. :)
Parts:
- removed R31, R36: 0, Resistor_SMD:R_0402_1005Metric, symbol Device:R
- R32, R37: value 150r -> 220R; footprint Resistor_SMD:R_0603_1608Metric -> Resistor_SMD:R_0805_2012Metric_Pad1.20x1.40mm_HandSolder; Package 0603 -> (none)
- R89: now not fitted; now left out of the parts list
Connections:
- net VIS_SW_G is gone; now on net GPIO03: Q6.1 (G)
- net GPIO04: now also Q7.1 (G), R89.2
