File: design/Page5.kicad_sch (KiCad schematic)
At the start: 9 parts, among them U1 74LVC1G126, U4 74LVC1G126

Commit message: updated, its functional, but needs routing finished. tweeks from Bornhack 2026 to be added. :)
Parts:
- removed C1, C2, C3: 1uF, Capacitor_SMD:C_0402_1005Metric, symbol Device:C
- removed D1: RB521S30T1G, jetson-nano-baseboard-footprints:SOD-523, symbol Device:D_Zener
- removed R8: 470K, Resistor_SMD:R_0402_1005Metric, symbol Device:R
- removed TP1: TestPoint, TestPoint:TestPoint_Pad_D2.0mm, symbol Connector:TestPoint
- removed U1, U4: 74LVC1G126, Package_TO_SOT_SMD:SOT-353_SC-70-5, symbol 74xGxx:74LVC1G126
Connections:
- net POWER_EN: no longer TP3.1
Other:
- note added: "Tie High remove gates"
