File: design/Page7.kicad_sch (KiCad schematic)
At the start: 1 part

Commit message: updated, its functional, but needs routing finished. tweeks from Bornhack 2026 to be added. :)
Parts:
- removed R13: 100k, Resistor_SMD:R_0402_1005Metric, symbol Device:R
- added D2: USBLC6-2SC6, Package_TO_SOT_SMD:SOT-23-6, symbol Power_Protection:USBLC6-2SC6
- added J1: USB_C_Receptacle, Connector_USB:USB_C_Receptacle_G-Switch_GT-USB-7010ASV, symbol Connector:USB_C_Receptacle
- added J7: USB_B_Micro, Connector_USB:USB_Micro-B_Amphenol_10103594-0001LF_Horizontal, symbol Connector:USB_B_Micro
- added R100, R101, R18: 5.1k, Resistor_SMD:R_0805_2012Metric_Pad1.20x1.40mm_HandSolder, symbol Device:R
Connections:
- net GND: now also D2.2 (GND), J1.A1 (GND), J1.A12 (GND), J1.B1 (GND), J1.B12 (GND), J1.S1 (SHIELD), J7.5 (GND), J7.6 (Shield), R100.2, R101.2, R18.2
- new net: J1.B5 (CC2), R100.1
- new net: J1.A5 (CC1), R101.1
- new net +5V: D2.5 (VBUS), J1.A4 (VBUS), J1.A9 (VBUS), J1.B4 (VBUS), J1.B9 (VBUS), J7.1 (VBUS)
- new net GPIO00: R18.1
- new net USB0_D_N: D2.3 (I/O2), D2.4 (I/O2), J1.A7 (D-), J1.B7 (D-), J7.2 (D-)
- new net USB0_D_P: D2.1 (I/O1), D2.6 (I/O1), J1.A6 (D+), J1.B6 (D+), J7.3 (D+)
- no-connect marks 0 -> 11
Other:
- note added: "ADD 5v power to VBUS control from GPIO, ask MAX"
- note added: "DEBUG MICRO USB CONNECTIONS"
- note added: "DNP for MPV"
- note added: "No stuff the common mode choke, co-locate resistors to avoid stubs"
- note added: "consider replacing with a usb c port for niceness."
- note added: "short to GND"
- note removed: "Level Shift for Servo PWM signal"
