File: design/Page4b.kicad_sch (KiCad schematic)
At the start: 8 parts, among them J5 2309414-1

Commit message: updated, its functional, but needs routing finished. tweeks from Bornhack 2026 to be added. :)
Parts:
- added D12, D13, D14, D15, D16, D17: TPD1E10B06DPYR, Diode_SMD:D_0402_1005Metric, symbol Device:D_TVS
- added J10: restart, Connector_PinSocket_2.54mm:PinSocket_2x01_P2.54mm_Vertical, symbol Connector:Conn_01x02_Pin
- added J13: recovery, Connector_PinSocket_2.54mm:PinSocket_2x01_P2.54mm_Vertical, symbol Connector:Conn_01x02_Pin
- added R8: 12k, Resistor_SMD:R_0805_2012Metric_Pad1.20x1.40mm_HandSolder, symbol Device:R
- R35: footprint Resistor_SMD:R_0402_1005Metric -> Resistor_SMD:R_0805_2012Metric_Pad1.20x1.40mm_HandSolder; Package 0402 -> (none)
Connections:
- net +5V: now also R8.1
- net FORCE_RECOVERY*: now also J13.2 (Pin_2)
- net I2C0_SCL: now also D14.1 (A1)
- net I2C0_SDA: now also D12.1 (A1)
- net I2C1_SCL: now also D13.1 (A1)
- net I2C1_SDA: now also D17.1 (A1)
- net I2C2_SCL: now also D15.1 (A1)
- net I2C2_SDA: now also D16.1 (A1)
- net POWER_EN: now also R8.2
- net SYS_RESET*: now also J10.2 (Pin_2)
- new net GND: D12.2 (A2), D13.2 (A2), D14.2 (A2), D15.2 (A2), D16.2 (A2), D17.2 (A2), J10.1 (Pin_1), J13.1 (Pin_1)
Other:
- note added: "DNP for MPV"
- note added: "remove and test."
- note removed: "Max says no place!"
- note removed: "max says have a mosfet controling this output, to prevent laod on the jetson pin."
- note removed: "no stuff option for debouncing"
