File: design/Page9.kicad_sch (KiCad schematic)
At the start: 8 parts, among them J3 SI-51005-F, J6 RJ45_RB1-125B8G1A, U3 Wurth_Magnetics_7490120110

Commit message: updated, its functional, but needs routing finished. tweeks from Bornhack 2026 to be added. :)
Parts:
- removed J3: SI-51005-F, jetson-nano-baseboard-footprints:SI-51005-F, symbol jetson-nano-baseboard:SI-51005-F
- removed R38: 220R, Resistor_SMD:R_0402_1005Metric, symbol jetson-nano-baseboard:R_220R_0402
- removed U3: Wurth_Magnetics_7490120110, FS-Magnetics:Wurth_749010012A, symbol FS-Ethernet:Wurth_Magnetics_7490120110
- added C1, C2: 0.1uF, Capacitor_SMD:C_0805_2012Metric_Pad1.18x1.45mm_HandSolder, symbol Device:C
- added C32, C33: 100pF, Capacitor_SMD:C_0805_2012Metric_Pad1.18x1.45mm_HandSolder, symbol jetson-nano-baseboard:C_100p_0402
- added D8: eth0, LED_SMD:LED_0603_1608Metric, symbol Device:LED
- added D9: eth1, LED_SMD:LED_0603_1608Metric, symbol Device:LED
- added J16: RJ45, Connector_RJ:RJ45_OST_PJ012-8P8CX_Vertical, symbol Connector:RJ45
- added J2: Serial-2, Connector_PinSocket_2.54mm:PinSocket_1x03_P2.54mm_Vertical, symbol Connector:Conn_01x03_Pin
- added Q1, Q2: DMN26D0UT-7, Package_TO_SOT_SMD:SOT-523, symbol Transistor_FET:2N7002
- added R10, R11, R31, R36: 75r, Resistor_SMD:R_0805_2012Metric_Pad1.20x1.40mm_HandSolder, symbol Device:R
- added R13, R15, R3, R9: 12k, Resistor_SMD:R_0805_2012Metric_Pad1.20x1.40mm_HandSolder, symbol Device:R
- added R39: 220R, Resistor_SMD:R_0805_2012Metric_Pad1.20x1.40mm_HandSolder, symbol jetson-nano-baseboard:R_220R_0402
- added TR1: G2415S, Transformer_Ethernet_HALO_TG111-MSC13, symbol Transformer:PT61020EL
- C4: renamed from C14; now not fitted; now left out of the parts list
- J6: now not fitted; now left out of the parts list
- R4, R5: Manufacturer Panasonic -> C25091; now not fitted; now left out of the parts list
- R40: footprint Resistor_SMD:R_0402_1005Metric -> Resistor_SMD:R_0805_2012Metric_Pad1.20x1.40mm_HandSolder; Manufacturer Panasonic -> C25091
Connections:
- net +3.3V: now also R39.2
- net ENET_LED0: now also D8.1 (K)
- net ENET_LED1: now also D9.1 (K)
- net ENET_TRD0_N: now also TR1.11 (TD4+)
- net ENET_TRD0_P: now also TR1.12 (TD4-)
- net ENET_TRD1_N: now also TR1.8 (TD3+)
- net ENET_TRD1_P: now also TR1.9 (TD3-)
- net ENET_TRD2_N: now also TR1.5 (TD2+)
- net ENET_TRD2_P: now also TR1.6 (TD2-)
- net ENET_TRD3_N: now also TR1.2 (TD1+)
- net ENET_TRD3_P: now also TR1.3 (TD1-)
- net GND: now also C1.2, C2.2, C32.2, C33.2, J2.1 (Pin_1)
- net at R40.2: now also D8.2 (A)
- new net: J2.3 (Pin_3), Q1.3 (D), R13.2
- new net: J2.2 (Pin_2), Q2.3 (D), R15.2
- new net: R31.1, TR1.21 (MCT2)
- new net: C32.1, R10.2, R11.2, R31.2, R36.2
- new net: C33.1, TR1.1 (TCT1), TR1.10 (TCT4), TR1.4 (TCT2), TR1.7 (TCT3)
- new net: R10.1, TR1.15 (MCT4)
- new net: R11.1, TR1.18 (MCT3)
- new net: R36.1, TR1.24 (MCT1)
- new net: D9.2 (A), R39.1
- new net +1V8: C1.1, Q1.1 (G), Q2.1 (G), R3.1, R9.1
- new net +3V3_HDMI: C2.1, R13.1, R15.1
- new net C1_N: J16.2, TR1.14 (MX4+)
- new net C1_P: J16.1, TR1.13 (MX4-)
- new net C2_N: J16.6, TR1.17 (MX3+)
- new net C2_P: J16.3, TR1.16 (MX3-)
- new net C3_N: J16.5, TR1.20 (MX2+)
- new net C3_P: J16.4, TR1.19 (MX2-)
- new net C4_N: J16.8, TR1.23 (MX1+)
- new net C4_P: J16.7, TR1.22 (MX1-)
- new net UART2_RXD: Q1.2 (S), R3.2
- new net UART2_TXD: Q2.2 (S), R9.2
- no-connect marks 2 -> 1
Other:
- note added: "B standard!"
- note added: "Brown"
- note added: "Corrected pinnout."
- note added: "DNP for MPV"
- note added: "FIX THIS MESS. SEE PHOTOS."
- note added: "Green"
- note added: "Orange"
- note added: "blue"
- note added: "https://www.lcsc.com/product-detail/C3003219.html"
- note added: "https://www.lcsc.com/product-detail/C7205130.html"

Commit message: cleaned up a bit, more to do
Parts:
- removed C4: 100pF, Capacitor_SMD:C_0402_1005Metric, symbol jetson-nano-baseboard:C_100p_0402
- removed J6: RJ45_RB1-125B8G1A, Connector_RJ:RJ45_UDE_RB1-125B8G1A, symbol Connector:RJ45_RB1-125B8G1A
- removed R4, R5: 220R, Resistor_SMD:R_0402_1005Metric, symbol jetson-nano-baseboard:R_220R_0402
- J2: now left out of the parts list
Connections:
- no-connect marks 1 -> 0
