File: design/Page13.kicad_sch (KiCad schematic)
At the start: 2 parts

Commit message: updated, its functional, but needs routing finished. tweeks from Bornhack 2026 to be added. :)
Parts:
- added C57, C58: 15pF, Capacitor_SMD:C_0805_2012Metric_Pad1.18x1.45mm_HandSolder, symbol Device:C
- added C59: 0.1uF, Capacitor_SMD:C_0805_2012Metric_Pad1.18x1.45mm_HandSolder, symbol Device:C
- added D4: BAS70-05, Package_TO_SOT_SMD:SOT-23, symbol CustomSymbols:BAS70-05
- added L2: 1.2nH, Inductor_SMD:L_0402_1005Metric, symbol Device:L
- added Q14: DMN26D0UT-7, Package_TO_SOT_SMD:SOT-523, symbol Transistor_FET:2N7002
- added Q8: MMBT3904, Package_TO_SOT_SMD:SOT-23, symbol Transistor_BJT:MMBT3904
- added R80: 36k, Resistor_SMD:R_0805_2012Metric_Pad1.20x1.40mm_HandSolder, symbol Device:R
- added R82, R83: 12k, Resistor_SMD:R_0805_2012Metric_Pad1.20x1.40mm_HandSolder, symbol Device:R
- R79: footprint Resistor_SMD:R_0402_1005Metric -> Resistor_SMD:R_0805_2012Metric
- R81: footprint Resistor_SMD:R_0402_1005Metric -> Resistor_SMD:R_0805_2012Metric_Pad1.20x1.40mm_HandSolder; Package 0402 -> (none)
Connections:
- net +3.3V: now also Q14.1 (G), R80.2
- net HDMI_CEC: now also D4.1 (A1), Q14.2 (S)
- net HDMI_HPD: now also Q8.3 (C)
- new net: D4.2 (A2), R80.1
- new net: D4.3 (C), L2.1, Q14.3 (D)
- new net: Q8.1 (B), R82.1, R83.2
- new net GND: C57.2, C58.2, C59.2, Q8.2 (E), R82.2
- new net HDMI_CEC_CON: C57.1, L2.2
- new net HDMI_HPD_CON: C58.1, C59.1, R83.1
Other:
- note added: "DNP for MPV"
- note added: "this is normaly high"
- moved on the sheet: R81

Commit message: updated little details.
Other:
- note added: "BJT to help with ESD COLD be the N mosfet"
Changed lines of the file:
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@@
+		)
+	)
+	(text "BJT to help with ESD\nCOLD be the N mosfet"
+		(exclude_from_sim no)
+		(at 48.26 157.734 0)
+		(effects
+			(font
+				(size 0.9906 0.9906)
+			)
 		)
 	)
