File: design/Page3.kicad_sch (KiCad schematic)
At the start: 4 parts, among them J5 2309414-1

Commit message: updated, its functional, but needs routing finished. tweeks from Bornhack 2026 to be added. :)
Parts:
- added C13, C14, C18, C19: 0.1uF, Capacitor_SMD:C_0402_1005Metric, symbol Device:C
- added C25, C26, C27, C28, C29, C3, C9: 100uF, Capacitor_SMD:C_0805_2012Metric_Pad1.18x1.45mm_HandSolder, symbol Device:C
- added D10: M.2, LED_SMD:LED_0603_1608Metric, symbol Device:LED
- added J15: Bus_M.2_Socket_M, Connector_PCBEdge:M.2_2280-xx-M, symbol Connector:Bus_M.2_Socket_M
- added JP1: DEVSLP, Jumper:SolderJumper-3_P1.3mm_Bridged2Bar12_Pad1.0x1.5mm_NumberLabels, symbol Jumper:SolderJumper_3_Bridged12
- added R6: 150r, Resistor_SMD:R_0603_1608Metric, symbol Device:R
- added R7: 12k, Resistor_SMD:R_0402_1005Metric, symbol Device:R
- C22, C23: footprint Capacitor_Tantalum_SMD:CP_EIA-3528-12_Kemet-T -> Capacitor_SMD:C_0805_2012Metric_Pad1.18x1.45mm_HandSolder
- C24: value 330uF -> 0.1uF; footprint Capacitor_SMD:C_Elec_6.3x7.7 -> Capacitor_SMD:C_0402_1005Metric; MPN TAJD337K010RNJ -> CL05B104KO5NNNC; Manufacturer TAJD337K010RNJ -> C1525; Package TAJD337K010RNJ -> 0402; Tolerance 20% -> 10%; now not fitted; now left out of the parts list
Connections:
- net +5V: now also C25.1, C26.1, C27.1, C28.1, C29.1, C3.1, C9.1; no longer C24.1
- net GND: now also C13.2, C14.2, C18.2, C19.2, C25.2, C26.2, C27.2, C28.2, C29.2, C3.2, C9.2, J15.1 (GND), J15.15 (GND), J15.21 (GND), J15.27 (GND), J15.3 (GND), J15.33 (GND), J15.39 (GND), J15.45 (GND), J15.51 (GND), J15.57 (GND), J15.71 (GND), J15.73 (GND), J15.75 (GND), J15.9 (GND), JP1.1 (A)
- net PCIE_Rx0_N: now reaches J5.131 (PCIE0_RX0_N)
- net PCIE_Rx0_N: now also J15.41 (PERn0/SATA-B+)
- net PCIE_Rx0_P: now reaches J5.133 (PCIE0_RX0_P)
- net PCIE_Rx0_P: now also J15.43 (PERp0/SATA-B-)
- net PCIE_Tx0_N: now reaches J5.134 (PCIE0_TX0_N)
- net PCIE_Tx0_N: now also J15.47 (PETn0/SATA-A-)
- net PCIE_Tx0_P: now reaches J5.136 (PCIE0_TX0_P)
- net PCIE_Tx0_P: now also J15.49 (PETp0/SATA-A+)
- net PCIE_Rx1_N: now reaches J5.137 (PCIE0_RX1_N)
- net PCIE_Rx1_N: now also J15.29 (PERn1)
- net PCIE_Rx1_P: now reaches J5.139 (PCIE0_RX1_P)
- net PCIE_Rx1_P: now also J15.31 (PERp1)
- net PCIE_Tx1_N: now reaches J5.140 (PCIE0_TX1_N)
- net PCIE_Tx1_N: now also J15.35 (PETn1)
- net PCIE_Tx1_P: now reaches J5.142 (PCIE0_TX1_P)
- net PCIE_Tx1_P: now also J15.37 (PETp1)
- net PCIE_Tx2_N: now reaches J5.148 (PCIE0_TX2_N)
- net PCIE_Tx2_N: now also J15.23 (PETn2)
- net PCIE_Rx2_N: now reaches J5.149 (PCIE0_RX2_N)
- net PCIE_Rx2_N: now also J15.17 (PERn2)
- net PCIE_Tx2_P: now reaches J5.150 (PCIE0_TX2_P)
- net PCIE_Tx2_P: now also J15.25 (PETp2)
- net PCIE_Rx2_P: now reaches J5.151 (PCIE0_RX2_P)
- net PCIE_Rx2_P: now also J15.19 (PERp2)
- net PCIE_Tx3_N: now reaches J5.154 (PCIE0_TX3_N)
- net PCIE_Tx3_N: now also J15.11 (PETn3)
- net PCIE_Rx3_N: now reaches J5.155 (PCIE0_RX3_N)
- net PCIE_Rx3_N: now also J15.5 (PERn3)
- net PCIE_Tx3_P: now reaches J5.156 (PCIE0_TX3_P)
- net PCIE_Tx3_P: now also J15.13 (PETp3)
- net PCIE_Rx3_P: now reaches J5.157 (PCIE0_RX3_P)
- net PCIE_Rx3_P: now also J15.7 (PERp3)
- net PCIE_CLK_N: now reaches J5.160 (PCIE0_CLK_N)
- net PCIE_CLK_N: now also J15.53 (REFCLKn)
- net PCIE_CLK_P: now reaches J5.162 (PCIE0_CLK_P)
- net PCIE_CLK_P: now also J15.55 (REFCLKp)
- net PCIE_WAKE: now reaches J5.179 (~{PCIE_WAKE})
- net PCIE_WAKE: now also J15.54 (~{PEWAKE})
- net PCIE_REQ: now reaches J5.180 (~{PCIE0_CLKREQ})
- net PCIE_REQ: now also J15.52 (~{CLKREQ})
- net PCIE_RST: now reaches J5.181 (~{PCIE0_RST})
- net PCIE_RST: now also J15.50 (~{PERST})
- new net: D10.1 (K), R6.1
- new net: J15.10 (DAS/~{DSS}/~{LED1}), R6.2
- new net: J15.38 (DEVSLP), JP1.2 (C)
- new net: J15.69 (PEDET), R7.2
- new net +1V8: D10.2 (A)
- new net +3.3V: C13.1, C14.1, C18.1, C19.1, C24.1, J15.12 (3.3V), J15.14 (3.3V), J15.16 (3.3V), J15.18 (3.3V), J15.2 (3.3V), J15.4 (3.3V), J15.70 (3.3V), J15.72 (3.3V), J15.74 (3.3V), JP1.3 (B), R7.1
- no-connect marks 69 -> 41
Other:
- note added: "NOT implemented in laybout."
- note added: "sets mode to sata (low) or PCI-E (high)"
- moved on the sheet: J5A

Commit message: added a 3 pin fan header PWM controlled of course.
Parts:
- added C4: 100uF, Capacitor_SMD:C_0805_2012Metric_Pad1.18x1.45mm_HandSolder, symbol Device:C
Connections:
- net +5V: now also C4.1
- net GND: now also C4.2
Changed lines of the file:
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@@
 	)
 	(junction
+		(at 334.01 80.01)
+		(diameter 0)
+		(color 0 0 0 0)
+	)
+	(junction
 		(at 109.22 92.71)
 		(diameter 0)
@@
 	)
 	(junction
+		(at 334.01 49.53)
+		(diameter 0)
+		(color 0 0 0 0)
+	)
+	(junction
 		(at 109.22 72.39)
 		(diameter 0)
@@
 	(wire
 		(pts
+			(xy 334.01 49.53) (xy 346.71 49.53)
+		)
+		(stroke
+			(width 0)
+			(type default)
+		)
+	)
+	(wire
+		(pts
 			(xy 308.61 49.53) (xy 308.61 54.61)
 		)
@@
 	(wire
 		(pts
+			(xy 346.71 80.01) (xy 346.71 62.23)
+		)
+		(stroke
+			(width 0)
+			(type default)
+		)
+	)
+	(wire
+		(pts
 			(xy -125.73 111.76) (xy -123.19 111.76)
 		)
@@
 	(wire
 		(pts
+			(xy 346.71 54.61) (xy 346.71 49.53)
+		)
+		(stroke
+			(width 0)
+			(type default)
+		)
+	)
+	(wire
+		(pts
 			(xy -6.35 102.87) (xy -6.35 105.41)
 		)
@@
 	(wire
 		(pts
+			(xy 334.01 80.01) (xy 346.71 80.01)
+		)
+		(stroke
+			(width 0)
+			(type default)
+		)
+	)
+	(wire
+		(pts
 			(xy 223.52 100.33) (xy 223.52 97.79)
 		)
@@
 					(unit 1)
 				)
+			)
+		)
+	)
+	(symbol
+		(lib_id "Device:C")
+		(at 346.71 58.42 0)
+		(unit 1)
+		(exclude_from_sim no)
+		(in_bom yes)
+		(on_board yes)
+		(dnp no)
+		(property "Reference" "C4"
+			(at 349.631 57.2516 0)
+			(effects
+				(font
+					(size 0.9906 0.9906)
+				)
+				(justify left)
+			)
+		)
+		(property "Value" "100uF"
+			(at 349.631 59.563 0)
+			(effects
+				(font
+					(size 0.9906 0.9906)
+				)
+				(justify left)
+			)
+		)
+		(property "Footprint" "Capacitor_SMD:C_0805_2012Metric_Pad1.18x1.45mm_HandSolder"
+			(at 347.6752 62.23 0)
+			(effects
+				(font
+					(size 1.27 1.27)
+				)
+				(hide yes)
+			)
+		)
+		(property "Datasheet" "~"
+			(at 346.71 58.42 0)
+			(effects
+				(font
+					(size 1.27 1.27)
+				)
+				(hide yes)
+			)
+		)
+		(property "Description" "C2286"
+			(at 346.71 58.42 0)
+			(effects
+				(font
+					(size 1.27 1.27)
+				)
+				(hide yes)
+			)
+		)
+		(property "Package" "CASE-B_3528"
+			(at 351.79 66.04 0)
+			(effects
+				(font
+					(size 0.9906 0.9906)
+				)
+			)
+		)
+		(property "Tolerance" "20%"
+			(at 351.79 68.58 0)
+			(effects
+				(font
+					(size 0.9906 0.9906)
+				)
+			)
+		)
+		(property "MPN" "T491B106M020AT"
+			(at 346.71 58.42 0)
+			(effects
+				(font
+					(size 1.27 1.27)
+				)
+				(hide yes)
+			)
+		)
+		(property "Manufacturer" "C2798040"
+			(at 346.71 58.42 0)
+			(effects
+				(font
+					(size 1.27 1.27)
+				)
+				(hide yes)
+			)
+		)
+		(pin "1"
+		)
+		(pin "2"
+		)
+		(instances
+			(project "baseboard"
+				(path "/dcdaf9eb-e0ef-4beb-9486-7183d93d6e4d/00000000-0000-0000-0000-00005ef2b870"
+					(reference "C4")
+					(unit 1)
+				)
