File: design/baseboard.kicad_pcb (KiCad board)
At the start: 2 copper layers, 88.2 x 86.9 mm, 132 parts, among them J1 USB_C_Receptacle, J10 restart, J11 HDMI_A, J12 USB3_A, J13 recovery, J16 RJ45, J2 Serial-2, J3 Jack-DC, J4 Conn_01x04_Male, J5 2309414-1, J8 power in, Q1 DMN26D0UT-7, Q11 DMN26D0UT-7, Q12 DMN26D0UT-7, Q13 DMN26D0UT-7, Q14 DMN26D0UT-7, Q2 DMN26D0UT-7, Q3 DMN26D0UT-7, Q4 DMN26D0UT-7, Q6 DMN26D0UT-7, Q7 DMN26D0UT-7, Q8 MMBT3904, U3 AMS1117-3.3, U4 AMS1117-1.8

Commit message: finished routing, doing some cleanup next.
Parts:
- moved D9 15.5 mm to (-9.09, 61.0)
- moved R39 15.5 mm to (-12.8, 61.3)
- moved C1 8.53 mm to (0.28, 79.9), turned to -90 degrees
- moved R35 6.82 mm to (6.12, 49.5), turned to 0 degrees
- moved R101 6.34 mm to (-12.7, 53.9)
- moved J16 5.19 mm to (-11.4, 66.3)
- moved J1 5.19 mm to (-20.4, 56.1)
- moved R100 4.75 mm to (-12.7, 57.2)
- moved D8 3.38 mm to (-9.06, 59.2)
- moved R40 3.33 mm to (-12.7, 59.2)
- moved J12 2.98 mm to (-12.2, 36.5)
- moved R15 2.28 mm to (-13.0, 81.2)
- moved Q1 2.26 mm to (3.62, 79.4)
- moved C32 2.16 mm to (-5.48, 74.9), turned to 90 degrees
- moved C2 1.83 mm to (3.51, 81.9)
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Routing:
- net ENET_LED1: track 57.8 -> 34.8 mm
- net +5V: track 310.7 -> 292.1 mm, vias 12 -> 11
- net +3.3V: track 373.2 -> 357.9 mm
- net /UART to USB Bridge/C2_N: track 6.26 -> 14.5 mm
- net /UART to USB Bridge/C3_N: track 6.85 -> 14.1 mm, vias 0 -> 2
- net /UART to USB Bridge/C3_P: track 5.21 -> 11.9 mm, vias 0 -> 2
- net GND: track 210.4 -> 204.6 mm, vias 177 -> 176
- net /UART to USB Bridge/C2_P: track 7.22 -> 12.8 mm, vias 0 -> 1
- net /UART to USB Bridge/C4_N: track 4.83 -> 9.72 mm
- net /UART to USB Bridge/C1_N: track 5.76 -> 10.3 mm
- net ENET_TRD3_N: track 21.9 -> 25.6 mm
- net ENET_TRD3_P: track 21.9 -> 25.5 mm
- net ENET_TRD2_P: track 20.5 -> 24.1 mm
- net ENET_TRD2_N: track 20.7 -> 24.2 mm
- net /UART to USB Bridge/C4_P: track 7.03 -> 10.2 mm
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Other:
- board text added: "compile 2 BOMbs - mvp ( power, SODIM, ethernet, fan) - mega ( power SODIM ethernet HDMI usb3 fan ) remove jumper, and unessaserry compenonets for cooling fan. as not needed."
- board text removed: "UART2 Rx"
- board text removed: "UART2 Tx"
- board text removed: "compile 2 BOMbs - mvp ( power, SODIM, ethernet, fan) - mega ( power SODIM ethernet HDMI usb3 fan ) finish routing ethernet. its corrected now, just need to flip the last 2 paris SPACE CONNECTORS APART. there kinda close, the USB and HDMI are too close, squeezing both in is a stress remove jumpter, as it worked as is. ????"

Commit message: cleaned up a bit, more to do
Parts:
- moved J11 0.79 mm to (-19.0, 19.4)
Routing:
- net +5V: track 292.1 -> 263.4 mm
- net /HDMI Connections Part 1/HDMI_TXC_CON_N: track 17.7 -> 18.5 mm
- net /HDMI Connections Part 1/HDMI_TX1_CON_N: track 17.5 -> 18.3 mm
- net /HDMI Connections Part 1/HDMI_TX0_CON_N: track 16.9 -> 17.7 mm
- net HDMI_HPD_CON: track 49.1 -> 49.9 mm
- net HDMI_CEC_CON: track 48.4 -> 49.2 mm
- net /HDMI Connections Part 1/HDMI_TXC_CON_P: track 17.7 -> 18.5 mm
- net /HDMI Connections Part 1/HDMI_TX2_CON_P: track 19.1 -> 19.8 mm
- net /HDMI Connections Part 1/HDMI_TX2_CON_N: track 18.9 -> 19.7 mm
- net /HDMI Connections Part 1/HDMI_TX1_CON_P: track 17.5 -> 18.3 mm
- net /HDMI Connections Part 1/HDMI_TX0_CON_P: track 16.7 -> 17.5 mm
- net /HDMI Connections Part 1/HDMI_DDC_SDA_POL_CON: track 14.1 -> 14.9 mm
- net /HDMI Connections Part 1/HDMI_DDC_SCL_POL_CON: track 10.6 -> 11.4 mm
- net GND: vias 176 -> 175
Other:
- board text added: "compile 2 BOMbs - mvp ( power, SODIM, ethernet, fan) - mega ( power SODIM ethernet HDMI usb3 fan ) remove jumper, and unessaserry compenonets for cooling fan. as not needed. simplifie BOM."
- board text removed: "compile 2 BOMbs - mvp ( power, SODIM, ethernet, fan) - mega ( power SODIM ethernet HDMI usb3 fan ) remove jumper, and unessaserry compenonets for cooling fan. as not needed."

Commit message: added a 3 pin fan header PWM controlled of course.
Parts:
- added C4: 100uF, Capacitor_SMD:C_0805_2012Metric_Pad1.18x1.45mm_HandSolder, F.Cu at (-4.25, 5.29)
- added J6: Conn_01x03_Pin, Connector_PinHeader_2.54mm:PinHeader_1x03_P2.54mm_Vertical, F.Cu at (1.67, -0.75)
- added Q5: DMN26D0UT-7, Package_TO_SOT_SMD:SOT-523, F.Cu at (43.8, 15.5)
- moved J8 14.3 mm to (-6.00, -0.28)
- moved C9 12.6 mm to (-7.00, 5.25), turned to -90 degrees
- moved J4 1.20 mm to (1.67, 4.00)
Routing:
- net Net-(J6-Pin_1): track 0.00 -> 63.0 mm, vias 0 -> 1
- net +5V: track 263.4 -> 257.8 mm
- net GND: track 204.6 -> 200.2 mm, vias 175 -> 178
- net /Power Regulation and Fan Tach/FAN_TACH_IN: track 51.8 -> 55.5 mm
- net /Power Regulation and Fan Tach/FAN_PWM_INV: track 4.25 -> 6.10 mm
- net /Power Regulation and Fan Tach/FAN_PWM_LS: track 46.0 -> 45.0 mm
- net Net-(D4-C): track 9.79 -> 8.80 mm
Other:
- outline, holes or cut-outs redrawn
- board text removed: "PWR"
